Commit message: v0 IA environnements

File: arduino_arm.urdf (robot description, URDF)
Before this commit: robot howtomechatronics_arm, 6 links, 5 joints
Links:
- removed link link_1
- removed link link_2
- removed link link_3
- removed link link_4
- added link forearm, mass 0.12; collision box size=0.025 0.03 0.12; collision box size=0.04 0.055 0.04
- added link gripper_base, mass 0.03; collision box size=0.023 0.032 0.012; collision box size=0.04 0.05 0.008
- added link gripper_left, mass 0.01; collision box size=0.008 0.005 0.015; collision box size=0.008 0.006 0.05
- added link gripper_right, mass 0.01; collision box size=0.008 0.005 0.015; collision box size=0.008 0.006 0.05
- added link rotating_base, mass 0.2; collision box size=0.05 0.06 0.04; collision cylinder length=0.02 radius=0.055
- added link upper_arm, mass 0.15; collision box size=0.03 0.035 0.13; collision box size=0.04 0.055 0.04
- added link wrist, mass 0.05; collision box size=0.023 0.032 0.023; collision box size=0.025 0.04 0.03
- link base_link: mass None -> 0.5; geometry collision cylinder length=0.005 radius=0.08; collision cylinder length=0.05 radius=0.065
- link tip: mass None -> 0.001
Joints:
- added joint joint_gripper_base: type fixed, parent wrist, child gripper_base, origin xyz=0 0 0.05 rpy=0 0 0
- added joint joint_gripper_left: type revolute, parent gripper_base, child gripper_left, origin xyz=0 0.015 0.02 rpy=0 0 0, axis 1 0 0, limit lower=0 upper=0.5 effort=5 velocity=1.0
- added joint joint_gripper_right: type revolute, parent gripper_base, child gripper_right, origin xyz=0 -0.015 0.02 rpy=0 0 0, axis 1 0 0, limit lower=-0.5 upper=0 effort=5 velocity=1.0
- joint joint_1: child link_1 -> rotating_base; limit lower=-1.57 upper=1.57 effort=10 velocity=1.0 -> lower=-2.618 upper=2.618 effort=10 velocity=1.0; origin xyz=0 0 0.04 rpy=0 0 0 -> xyz=0 0 0.05 rpy=0 0 0
- joint joint_2: child link_2 -> upper_arm; parent link_1 -> rotating_base
- joint joint_3: child link_3 -> forearm; parent link_2 -> upper_arm
- joint joint_4: child link_4 -> wrist; limit lower=-1.57 upper=1.57 effort=10 velocity=1.0 -> lower=-1.57 upper=1.57 effort=5 velocity=1.0; parent link_3 -> forearm
- joint joint_tip: origin xyz=0 0 0.11 rpy=0 0 0 -> xyz=0 0 0.07 rpy=0 0 0; parent link_4 -> gripper_base
